File: DIY amplifier.kicad_pcb (KiCad board)
At the start: 4 copper layers, 90.9 x 71.6 mm, 87 parts, among them J1 AudioPlug3, J2 Output, J3 Input, Q1 IRF540N, Q2 IRF540N, Q3 IRF540N, Q4 IRF540N, Q5 DMN2310U, Q6 BC858, Q7 BC858, Q8 BC848, Q9 BC858, SW1 Reset, U1 74LVC1G14, U10 INA181, U11 74LVC2G17, U2 OPA310SxDBV, U3 HIP4081A, U4 74LVC1G17, U5 L7805, U6 L7812, U7 TLV3501AIDBV, U8 MCP6561U

Commit message: Add files via upload
Parts:
- added C24: 0.1u, Capacitor_SMD:C_0402_1005Metric, B.Cu at (44.0, 45.4)
- added Q10: PJA3431, Package_TO_SOT_SMD:SOT-23-3, B.Cu at (41.3, 49.8)
- added R30: 10k, Resistor_SMD:R_0603_1608Metric, B.Cu at (44.2, 49.5)
- added U9: 74LVC1G17, Package_TO_SOT_SMD:SOT-23-5, B.Cu at (32.9, 47.9)
- SW1: value Reset -> SW_Push
- U11: value 74LVC2G17 -> 74LVC1G14; footprint Package_TO_SOT_SMD:SOT-363_SC-70-6 -> Package_TO_SOT_SMD:SOT-23-5
- moved C10 12.8 mm to (30.6, 48.6), turned to 90 degrees
- moved R9 12.3 mm to (60.8, 37.0), turned to 0 degrees
- moved R26 10.9 mm to (34.0, 50.8), turned to 180 degrees
- moved R16 8.39 mm to (86.2, 31.7), turned to 90 degrees
- moved SW1 5.82 mm to (30.6, 41.4), turned to 90 degrees
- moved R24 5.60 mm to (39.7, 44.9), turned to 0 degrees
- moved Q9 5.48 mm to (37.3, 49.9), turned to -90 degrees
- moved R20 5.21 mm to (63.1, 61.2), turned to 0 degrees
- moved Q8 4.56 mm to (36.4, 45.8), turned to 90 degrees
- moved R25 3.09 mm to (39.7, 46.9), turned to 0 degrees
- moved U11 2.95 mm to (43.4, 43.1)
- moved C11 2.16 mm to (67.6, 23.0)
- moved C21 2.16 mm to (70.0, 25.5)
- moved C20 1.13 mm to (82.6, 25.2)
- moved C18 1.13 mm to (80.1, 22.7)
Connections:
- R24 pad 2: Net-(SW1-A) -> Net-(Q10-D)
- R25 pad 2: Net-(SW1-A) -> Net-(Q10-D)
- SW1 pad 1: Net-(SW1-A) -> +5V
- SW1 pad 2: +5V -> Net-(Q10-G)
- U11 pad 1: Net-(U10-Pad1) -> unconnected-(U11-NC-Pad1)
- U11 pad 2: GND -> Net-(Q8-C)
- U11 pad 3: Net-(Q8-C) -> GND
Routing:
- net Net-(Q10-G): track 0.00 -> 25.5 mm, vias 0 -> 1
- net Net-(SW1-A): track 13.2 -> 0.00 mm
- net GND: track 98.8 -> 110.4 mm, vias 17 -> 14
- net Net-(U10-Pad1): track 21.5 -> 29.8 mm, vias 0 -> 2
- net +5V: track 43.4 -> 51.0 mm, vias 10 -> 11
- net Net-(Q2-G): track 25.8 -> 31.9 mm
- net Net-(Q10-D): track 0.00 -> 5.30 mm
- net A out: track 60.6 -> 56.5 mm
- net Vcc: track 0.00 -> 3.74 mm
- net Net-(Q8-C): track 9.09 -> 11.3 mm
- net Net-(R26-Pad2): track 3.72 -> 2.00 mm
- net Net-(Q1-G): track 15.6 -> 14.0 mm
- net DIS: track 7.91 -> 9.29 mm
- net R_shunt: track 117.6 -> 116.8 mm
- net B out: track 70.1 -> 69.4 mm
Other:
- board text added: "Input : 15-35V Output : 4Ω, 6A"
